File: rpib big shield/shield.brd (EAGLE design)
At the start: 100 x 73.3 mm, 23 parts, among them IC1 DS2482-100S, IC2 AT24C, IC4 DS18B20, U1 DS1307ZN+, U3 AT32UC3L016-AUT, X1 MSTBA4

Commit message: asd
Parts:
- removed JP5: (no value), pinhead:1X05
- added JP3: (no value), pinhead:2X20
- added JP4: (no value), pinhead:1X08/90
- added SV4, SV5: (no value), X_Pfostenstecker:ML10
- JP7: device pinhead:2X03 -> pinhead:1X06/90
- moved CN1 76.6 mm to (96.5, 12.7)
- moved X1 51.5 mm to (77.5, 75.6), turned to 180 degrees
- moved R2 39.4 mm to (20.3, 54.6), turned to 270 degrees
- moved BAT1 33.1 mm to (45.7, 34.9)
- moved IC2 32.4 mm to (26.7, 55.2)
- moved ZD1 31.6 mm to (87.6, 29.8), turned to 270 degrees
- moved U$1 28.6 mm to (55.2, 48.3), turned to 180 degrees
- moved JP7 27.9 mm to (99.7, 35.6), turned to 270 degrees
- moved U3 27.3 mm to (6.99, 43.2)
- moved U1 26.2 mm to (54.0, 54.6), turned to 90 degrees
- moved JP2 24.2 mm to (26.7, 49.5), turned to 180 degrees
- moved IC1 20.7 mm to (77.5, 29.8)
- moved C2 14.2 mm to (31.1, 36.2)
- moved C3 14.2 mm to (26.7, 31.8)
- moved U$2 14.2 mm to (26.7, 36.2)
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Connections:
- removed net N$10: JP7.5, JP7.6, ZD1.5
- removed net N$7: JP5.3
- removed net N$8: JP5.4
- removed net N$9: JP7.3, JP7.4, ZD1.6
- new net 3V3@2: JP3.17, PCB1.17
- net 1WIRE_DATA: now also JP3.7
- net BUTTON_DOWN: now also JP3.18
- net BUTTON_ENCODER_MENUE: now also JP3.37
- net BUTTON_NEXT: now also JP3.40
- net BUTTON_PAUSE: now also JP3.12
- net BUTTON_PLAY: now also JP3.16
- net BUTTON_PREV: now also JP3.38
- net BUTTON_UP: now also JP3.22
- net BUTTON_VOL_DOWN: now also JP3.24
- net BUTTON_VOL_UP: now also JP3.32
- net ENCODER_1: now also JP3.33
- net ENCODER_2: now also JP3.35
- net GND: now also JP3.14, JP3.20, JP3.30, JP3.34, JP3.6, JP4.1, JP4.2, SV5.2; no longer JP5.5
- net GND@1: now also JP3.25, JP3.39, JP3.9
- net HALTE_RELAI: now also JP3.29, JP4.5, JP4.6
- net ID_SC: now also JP3.28
- net ID_SD: now also JP3.27
- net LED0: now also JP3.11
- net LED1: now also JP3.13
- net LED_LAN_RUN: now also JP3.31
- net LED_STATUS: now also JP3.36
- net MISO: now also JP3.21, SV5.7
- net MOSI: now also JP3.19, SV5.8
- net N$2: now also JP7.3, JP7.6, ZD1.5; no longer JP5.1
- net N$6: now also JP7.2, JP7.5, ZD1.6; no longer JP5.2
- net P3V3: now also JP3.1, JP7.1, JP7.4, SV5.1
- net P5V: now also JP3.2, JP3.4, JP4.7, JP4.8
- net RPI_RX: now also JP3.10, SV5.3
- net RPI_TX: now also JP3.8, SV5.4
- net SCK: now also JP3.23, SV5.9
- net SCL: now also JP3.5, SV5.5
- net SDA: now also JP3.3, SV5.6
- net SSEL: now also JP3.26, SV5.10
- net ZUENDPLUS_LED2: now also JP3.15, JP4.3, JP4.4
Routing:
- net SCL: track 0.00 -> 71.2 mm, vias 0 -> 1
- net SDA: track 0.00 -> 64.1 mm, vias 0 -> 2
- net MISO: track 0.00 -> 47.7 mm, vias 0 -> 1
- net SCK: track 0.00 -> 46.3 mm, vias 0 -> 1
- net MOSI: track 0.00 -> 44.7 mm, vias 0 -> 2
- net RPI_RX: track 0.00 -> 42.5 mm, vias 0 -> 1
- net GND: track 0.00 -> 41.9 mm
- net RPI_TX: track 0.00 -> 39.5 mm, vias 0 -> 1
- net SSEL: track 0.00 -> 38.3 mm, vias 0 -> 2
- net 1WIRE_DATA: track 0.00 -> 37.1 mm
- net GND@1: track 0.00 -> 33.7 mm
- net P3V3: track 0.00 -> 28.6 mm
- net N$2: track 0.00 -> 19.4 mm
- net N$6: track 0.00 -> 17.6 mm
- net ID_SD: track 0.00 -> 16.2 mm
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- added copper zone on layer 1, net GND
Other:
- board size 100 x 73.3 mm -> 100 x 100 mm
- board text added: "ENC/LED"
- board text removed: "ENC"
- board text removed: "RTC"
- board text removed: "RTC BATT"
- board text removed: "UEXT"
