File: rpib big shield/shield.sch (EAGLE design)
At the start: 23 parts, among them IC1 DS2482-100S, IC2 AT24C, IC4 DS18B20, U1 DS1307ZN+, U3 AT32UC3L016-AUT, X1 MSTBA4

Commit message: asd
Parts:
- removed JP5: (no value), pinhead:PINHD-1X5
- added JP3: (no value), pinhead:PINHD-2X20
- added JP4: (no value), pinhead:PINHD-1X8/90
- added SV4, SV5: (no value), X_Pfostenstecker:ML10
- JP7: device pinhead:PINHD-2X3 -> pinhead:PINHD-1X6/90
Connections:
- removed net N$10: JP7.5, JP7.6, ZD1.P$3
- removed net N$7: JP5.3
- removed net N$8: JP5.4
- removed net N$9: JP7.3, JP7.4, ZD1.P$4
- new net 3V3@2: JP3.17, PCB1.3V3@2
- net 1WIRE_DATA: now also JP3.7
- net BUTTON_DOWN: now also JP3.18
- net BUTTON_ENCODER_MENUE: now also JP3.37
- net BUTTON_NEXT: now also JP3.40
- net BUTTON_PAUSE: now also JP3.12
- net BUTTON_PLAY: now also JP3.16
- net BUTTON_PREV: now also JP3.38
- net BUTTON_UP: now also JP3.22
- net BUTTON_VOL_DOWN: now also JP3.24
- net BUTTON_VOL_UP: now also JP3.32
- net ENCODER_1: now also JP3.33
- net ENCODER_2: now also JP3.35
- net GND: now also JP3.14, JP3.20, JP3.30, JP3.34, JP3.6, JP4.1, JP4.2, SV5.2; no longer JP5.5
- net GND@1: now also JP3.25, JP3.39, JP3.9
- net HALTE_RELAI: now also JP3.29, JP4.5, JP4.6
- net ID_SC: now also JP3.28
- net ID_SD: now also JP3.27
- net LED0: now also JP3.11
- net LED1: now also JP3.13
- net LED_LAN_RUN: now also JP3.31
- net LED_STATUS: now also JP3.36
- net MISO: now also JP3.21, SV5.7
- net MOSI: now also JP3.19, SV5.8
- net N$2: now also JP7.3, JP7.6, ZD1.P$3; no longer JP5.1
- net N$6: now also JP7.2, JP7.5, ZD1.P$4; no longer JP5.2
- net P3V3: now also JP3.1, JP7.1, JP7.4, SV5.1
- net P5V: now also JP3.2, JP3.4, JP4.7, JP4.8
- net RPI_RX: now also JP3.10, SV5.3
- net RPI_TX: now also JP3.8, SV5.4
- net SCK: now also JP3.23, SV5.9
- net SCL: now also JP3.5, SV5.5
- net SDA: now also JP3.3, SV5.6
- net SSEL: now also JP3.26, SV5.10
- net ZUENDPLUS_LED2: now also JP3.15, JP4.3, JP4.4
Other:
- note added: "Encoder/LED"
- note added: "Gyro"
- note added: "ID_EEPROM"
- note added: "UEXT/ATMEGA"
- note added: "UEXT/RPI"
- note removed: "Dreh Encoder"
- note removed: "UEXT"
