File: rpib big shield/Neuer Ordner/shield.sch (EAGLE design)
At the start: 42 parts, among them IC1 DS2482-100S, IC2 AT24C, IC3 SAMD21G18A-AUT, IC4 DS18B20, IC5 LT1615, U1 DS1307ZN+, X1 MSTBA4

Commit message: lipo charger and Sepic
Parts:
- removed C4: 4µ7 10V, MYPASS:CAP0805
- removed C5: 1µ, MYPASS:CAP0805
- removed C6: 10µ 5V, MYPASS:CAP0805
- removed C7: 4p7, mypassive-bleifrei:CAP0603R
- removed D1: MBR0520L, MYDISCR:MBR0520L
- removed IC5: LT1615, MYLT:LT1615
- removed JP5: (no value), schlager_modules:GY-521
- removed JP6: (no value), pinhead:PINHD-2X3
- removed L1, L2: 744032100, myinductiv:WE-LQ
- removed R3: 1M, mypassive-bleifrei:RES0603R
- added L6: MH2029-300Y, Protezione:0001_BLM21PG300SN1D_/_MH2029-300Y
- added R15: 10k, schlager_passiv:R-EU_R0805
- R1: value 604K -> 10k; device mypassive-bleifrei:RES0603R -> schlager_passiv:R-EU_R0805
Connections:
- net ID_SCL renamed ID_SC
- net ID_SDA renamed ID_SD
- net RPI_MISO renamed MISO
- net RPI_MOSI renamed MOSI
- net RPI_SCK renamed SCK
- removed net 12V: JP4.7, JP4.8, X1-1.1
- removed net ASDFASDASD: JP4.3, JP4.4, X1-3.1
- removed net FONA_RESET: JP1.5
- removed net FONA_RX: JP1.10
- removed net FONA_TX: JP1.9
- removed net GND_KFZ: JP4.1, JP4.2, X1-4.1
- removed net N$10: IC1G$1.1W, ZD1.P$1
- removed net N$16: C7.1, IC5.FB, R1.2, R3.1
- removed net N$7: C5.2, IC5.SW, L1.P$2
- removed net N$8: C5.1, D1.A, L2.P$1
- removed net N$9: C6.2, C7.2, D1.K, JP6.3, R3.2
- removed net PBAT: C4.2, IC5./SHDN, IC5.VIN, JP1.1, L1.P$1
- removed net RPI_1WIRE: IC4_1W.1W, JP3.7, PCB1.GPIO4/GCKL
- removed net RPI_SCL: IC1G$1.SCL, JP3.5, JP5.3, PCB1.GPIO3/SCL1, SV2.5, SV3.5, SV5.5, U$2.SCL, U1.SCL
- removed net RPI_SDA: IC1G$1.SDA, JP3.3, JP5.4, PCB1.GPIO2/SDA1, SV2.6, SV3.6, SV5.6, U$2.SDA, U1.SDA
- removed net ZUEND_KFZ: JP4.5, JP4.6, X1-2.1
- new net 1WIRE_DATA: IC1G$1.1W, IC4_1W.1W, JP3.7, PCB1.GPIO4/GCKL, ZD1.P$1
- new net CS_MCP: IC3.PA18/EIC/SCOM1PAD2+/TC3
- new net DGI_GPIO0: IC3.PA13/I2C/EIC/SCOM2PAD1+/TC2
- new net DGI_GPIO1: IC3.PA21/EIC/SCOM5PAD3+
- new net DGI_GPIO2: IC3.PA6/EIC/AIN6/SCOM0PAD2/TC1
- new net N$15: C22.1, IC3.VDDANA, L6.1
- new net PA00_XIN32: IC3.PA0/XIN32/EIC/SCOM1PAD0/TC2
- new net PA01_XOUT32: IC3.PA1/XOUT32/EIC/SCOM1PAD1/TC2
- new net PA03_AREFA: IC3.PA3/EIC/REF/AIN1
- new net PA08_TCC0-W0: IC3.PA8/I2C/AIN16/SCOM2PAD0+/TC0
- new net PA10_TCC0-W2: IC3.PA10/EIC/AIN18/SCOM2PAD2+/TC1
- new net PA11_TCC0-W3: IC3.PA11/EIC/AIN19/SCOM2PAD3+/TC1
- new net PA20_TCC0-W6: IC3.PA20/EIC/SCOM5PAD2+
- new net PA27_TX_LED: IC3.PA27/EIC
- new net PA28_USB_HOST_EN: IC3.PA28/EIC
- new net PB02_AIN10: IC3.PB2/EIC/AIN10/SCOM5PAD0
- new net PB03_RX_LED: IC3.PB3/EIC/AIN11/SCOM5PAD1
- new net PB10_S4_SPI_MOSI: IC3.PB10/EIC/SCOM4PAD2/TC5
- new net PB11_S4_SPI_SCK: IC3.PB11/EIC/SCOM4PAD3/TC5
- new net PB12_S4_SPI_MISO: IC3.PA12/I2C/EIC/SCOM2PAD0+/TC2
- new net SCL: IC1G$1.SCL, IC3.PA23/I2C/EIC/SCOM5PAD1+/TC4, JP3.5, PCB1.GPIO3/SCL1, R1.1, SV2.5, SV3.5, SV5.5, U$2.SCL, U1.SCL
- new net SDA: IC1G$1.SDA, IC3.PA22/I2C/EIC/SCOM5PAD0+/TC4, JP3.3, PCB1.GPIO2/SDA1, R15.1, SV2.6, SV3.6, SV5.6, U$2.SDA, U1.SDA
- net +3V3: now also L6.2, R1.2, R15.2; no longer C22.1, IC3.VDDANA, JP6.2, JP6.4
- net GND: now also JP4.1, JP4.2, X1-4.1; no longer C4.1, C6.1, IC5.GND, JP1.2, JP1.7, JP5.2, L2.P$2, R1.1, U$2.AD0
- net HALTE_RELAI: now also JP4.5, JP4.6, X1-2.1
- net P3V3: no longer JP5.1, JP6.1
- net P5V: now also JP4.7, JP4.8, X1-1.1
- net ZUENDPLUS_LED2: now also JP4.3, JP4.4, X1-3.1
Other:
- note added: "UEXT/ATMEGA"
- note removed: "UEXT/GPS"
- note removed: "UEXT/LCD"
