File: Baseboard/shield.sch (EAGLE design)
At the start: 54 parts, among them CON1 B2BPHSM, CON2 B2BPHSM, IC1 DS2482-100S, IC2 AT24C, IC3 MCP73871, IC4 DS18B20, Q1 MMUN2133LT1G, U1 DS1307ZN+, U2 TPS61090RSAR

Commit message: unknown old changes
Parts:
- removed C10, C8, C9: 4µ7, schlager_passiv:C-EUC1206
- removed C11: 10uF, schlager_passiv:C-EUC1206
- removed C12: 2.2uF, schlager_passiv:C-EUC1206
- removed C13: 0.1uF, schlager_passiv:C-EUC1206
- removed C15: 100uf/6v, schlager_passiv:CPOL-EUB/3528-21W
- removed CN1: (no value), adafruit:USBMINIB
- removed CON1, CON2: B2BPHSM, CAB:B2BPHSM
- removed IC4: DS18B20, 1wire:DS18B20
- removed JP1, JP2: (no value), pinhead:PINHD-1X2
- removed JP5: (no value), schlager_modules:GY-521
- removed L4: WE-HCC_8070, Wuerth_Elektronik_eiSos_V6:WE-HCC_8070
- removed LBO: RED, microbuilder:LED0805_NOOUTLINE
- removed LED1, LED2, LED3, LED4: (no value), led:LEDCHIP-LED0805
- removed PWR: GREEN, microbuilder:LED0805_NOOUTLINE
- removed R10, R8, R9: 1k, schlager_passiv:R-EU_R1206
- removed R15, R21: 1K, schlager_passiv:R-EU_R1206
- removed R16, R19: 340K, schlager_passiv:R-EU_R1206
- removed R17, R20: 1.87Mohm, schlager_passiv:R-EU_R1206
- removed R18: 200K, schlager_passiv:R-EU_R1206
- removed R4: 3k3, schlager_passiv:R-EU_R1206
- removed R5: 200k, schlager_passiv:R-EU_R1206
- removed R6: 18k, schlager_passiv:R-EU_R1206
- removed R7: 47k, schlager_passiv:R-EU_R1206
- removed R99: (no value), schlager_passiv:R-EU_R1206
- removed SV1: (no value), X_Pfostenstecker:ML16L
- removed SV3: (no value), X_Pfostenstecker:ML10L
- removed U2: TPS61090RSAR, microbuilder:VREG_TPS6103X
- added BAT1: (no value), con_bat_2032__s_:CR2032
- added C4, C5: (no value), schlager_passiv:CPOL-EUE5-13
- added F1: FUSEBLANK_5X20MM, fuse:FUSEBLANK_5X20MM
- added K1, K3: G5LE, relay:G5LE
- added MOD1: (no value), kim055l:KIM-055L
- added SJ1: (no value), jumper:SJM
- added SV2: (no value), X_Pfostenstecker:ML10
- added U$4: 1N4004, diode:1N4004
- added U3: (no value), adafruit:GPS_FGPMMOPA6H
- added X2: MSTBA3, X_Phoenix:MSTBA3
- IC3: value MCP73871 -> DS18B20; device MYMCHIP:MCP73871 -> 1wire:DS18B20
- JP7: device pinhead:PINHD-1X3 -> pinhead:PINHD-2X3/90
- Q1: value MMUN2133LT1G -> BC547; device transistor:MUN2114T1-PNP_DRIVER-SC59-BEC -> transistor-npn:BC547
- R1: value 1k -> 15k; device schlager_passiv:R-EU_R1206 -> schlager_passiv:R-EU_0207/7
Connections:
- net ID_SCL renamed ID_SC
- net ID_SDA renamed ID_SD
- net LCD_TP_IRQ renamed LED0
- removed net ENABLE: R16.2, U2.EN
- removed net ENCODDER_2: SV1.11
- removed net LBO: Q1.B, U2.LBO
- removed net LCD_CS: PCB1.!CE0!/GPIO8
- removed net LCD_RESET: PCB1.GEN/6GPIO25
- removed net LCD_RS: PCB1.GEN5/GPIO24
- removed net LCD_TS_CS: PCB1.!CE!/GPIO7, SV3.10
- removed net N$12: IC3.THERM, R99.2
- removed net N$13: IC3.PROG1, R4.2
- removed net N$14: IC3.PROG3, R5.2
- removed net N$15: IC3.VPCC, R6.2, R7.1
- removed net N$17: LED2.A, R8.1
- removed net N$18: LED3.A, R9.1
- removed net N$19: LED4.A, R10.1
- removed net N$20: IC3.STAT1/LBO, LED4.C
- removed net N$21: IC3.STAT2, LED3.C
- removed net N$22: IC3./PG, LED2.C
- removed net N$23: R19.2, R20.1, U2.LBI
- removed net N$24: PWR.C, R15.1
- removed net N$25: R17.1, R18.2, U2.FB
- removed net N$26: LBO.A, R21.1
- removed net N$27: Q1.C, R21.2
- removed net PBAT: C11.1, C13.1, C9.2, CON2.2, IC3.VBAT, L4.1, R20.2, U2.VBAT
- removed net PUSB: C8.2, CN1.VBUS, IC3.CE, IC3.IN, JP1.2, R10.2, R7.2, R8.2, R9.2
- removed net RPI_1WIRE: IC4_1W.1W, PCB1.GPIO4/GCKL
- removed net RPI_MISO: PCB1.GPIO9/MISO, SV3.7
- removed net RPI_MOSI: PCB1.GPIO10/MOSI, SV3.8
- removed net RPI_SCK: PCB1.GPIO11/SCLK, SV3.9
- removed net RPI_SCL: IC1G$1.SCL, JP5.3, PCB1.GPIO3/SCL1, SV3.5, U$2.SCL, U1.SCL
- removed net RPI_SDA: IC1G$1.SDA, JP5.4, PCB1.GPIO2/SDA1, SV3.6, U$2.SDA, U1.SDA
- removed net STATUS_LED: LED1.C, PCB1.GPIO18
- removed net VBAT: Q1.E, R16.1
- new net 12V: C4.+, K12.S, K32.S, MOD1.V+IN
- new net 1WIRE_DATA: IC1G$1.1W, IC3_1W.1W, PCB1.GPIO4/GCKL, ZD1.P$1
- new net GND@1: PCB1.GND@1, PCB1.GND@2, PCB1.GND@3
- new net GND_KFZ: K11.2, X2-2.1
- new net HALTE_RELAI: PCB1.GPIO5, R1.1
- new net LED1: PCB1.GPIO27/GEN2
- new net LED_LAN_RUN: PCB1.GPIO6
- new net LED_STATUS: PCB1.GPIO16
- new net MISO: PCB1.GPIO9/MISO, SV2.7
- new net MOSI: PCB1.GPIO10/MOSI, SV2.8
- new net POWER_KFZ: F1.2, K12.P, K32.P
- new net SCK: PCB1.GPIO11/SCLK, SV2.9
- new net SCL: IC1G$1.SCL, PCB1.GPIO3/SCL1, SV2.5, U$2.SCL, U1.SCL
- new net SDA: IC1G$1.SDA, PCB1.GPIO2/SDA1, SV2.6, U$2.SDA, U1.SDA
- new net SSEL: PCB1.!CE!/GPIO7, SV2.10
- new net ZUENDPLUS_LED2: PCB1.GPIO22/GEN3
- new net ZUEND_KFZ: K11.1, X2-3.1
- net BUTTON_DOWN: now also PCB1.GEN5/GPIO24; no longer PCB1.GPIO5, SV1.7
- net BUTTON_ENCODER_MENUE: now also PCB1.GPIO26; no longer PCB1.GPIO20, SV1.4
- net BUTTON_NEXT: now also PCB1.GPIO21; no longer PCB1.GPIO6, SV1.5
- net BUTTON_PAUSE: now also PCB1.GPIO18; no longer PCB1.GPIO12, SV1.8
- net BUTTON_PLAY: now also PCB1.GEN4/GPIO23; no longer PCB1.GPIO13, SV1.6
- net BUTTON_PREV: now also PCB1.GPIO20; no longer PCB1.GPIO16, SV1.3
- net BUTTON_UP: now also PCB1.GEN/6GPIO25; no longer PCB1.GPIO22/GEN3, SV1.9
- net BUTTON_VOL_DOWN: now also PCB1.!CE0!/GPIO8; no longer PCB1.GPIO21, SV1.2
- net BUTTON_VOL_UP: now also PCB1.GPIO12; no longer PCB1.GPIO26, SV1.1
- net ENCODER_1: now also PCB1.GPIO13; no longer PCB1.GEN4/GPIO23, SV1.10
- net GND: now also BAT1.NEG, C4.-, C5.-, IC3P.GND, MOD1.GNDIN, MOD1.GNDOUT, Q1.E, SJ1.2, SV2.2, U3.GND@1, U3.GND@2, U3.GND@3, U3.GND@4; no longer C10.1, C11.2, C12.2, C13.2, C15.-, C8.1, C9.1, CN1.GND, CON1.2, CON2.1, IC3./TE, IC3.GND, IC3.SEL, IC4P.GND, JP2.1, JP5.2, LBO.C, PCB1.GND@1, PCB1.GND@2, PCB1.GND@3, R15.2, R18.1, R19.1, R4.1, R5.1, R6.1, R99.1, SV1.16, SV3.2, U$2.AD0, U2.GND, U2.PGND, U2.SYNC
- net N$1: now also BAT1.POS2; no longer CON1.1
- net N$10: now also JP7.5, JP7.6, ZD1.P$3; no longer IC1G$1.1W, ZD1.P$1
- net N$2: now also K31.2, Q1.C, U$4.A; no longer JP7.3, ZD1.P$3
- net N$5: now also SJ1.1; no longer JP2.2
- net N$6: now also Q1.B, R1.2; no longer JP7.2, ZD1.P$4
- net N$7: now also F1.1, X2-1.1; no longer LED1.A, R1.1
- net N$9: now also JP7.3, JP7.4, ZD1.P$4; no longer L4.2, U2.SW
- net P3V3: now also IC3P.VDD, SV2.1, U3.VBACKUP, U3.VCC; no longer IC4P.VDD, JP5.1, JP7.1, R1.2, SV3.1, U1.VCC
- net P5V: now also C5.+, K31.1, MOD1.V+OUT1, MOD1.V+OUT2, U$4.C, U1.VCC; no longer C10.2, C12.1, C15.+, IC3.OUT, IC3.PROG2, JP1.1, PWR.A, R17.2, U2.VOUT
- net RPI_RX: now also SV2.3, U3.TX; no longer SV3.3
- net RPI_TX: now also SV2.4, U3.RX; no longer SV3.4
Other:
- note added: "UEXT"
- note removed: "4,5V"
- note removed: "6.8uH power w/2A current"
- note removed: "Buttons"
- note removed: "Gyro"
- note removed: "ID_EEPROM"
- note removed: "R2 < 500K R1 = 5.5*R2 (3.2V LBO)"
- note removed: "See Pg 15 1st para"
- note removed: "UEXT/LCD"
